Commit message: Modified some parameters

File: hector_quadrotor/hector_quadrotor_description/urdf/quadrotor_with_stereo_cam_with_IMU.gazebo.xacro (robot description, xacro)
@@ -14,5 +14,5 @@
         <topicName>imu</topicName>
         <bodyName>imu_link</bodyName>
-        <updateRateHZ>10.0</updateRateHZ>
+        <updateRateHZ>200.0</updateRateHZ>
         <gaussianNoise>0.0</gaussianNoise>
         <xyzOffset>0 0 0</xyzOffset>

File: hector_quadrotor/hector_quadrotor_description/urdf/quadrotor_with_stereo_cam_with_IMU.urdf.xacro (robot description, xacro)
@@ -8,6 +8,6 @@
     <!-- Stereo camera -->
     <xacro:include filename="$(find hector_sensors_description)/urdf/generic_stereo_camera.urdf.xacro" />
-    <xacro:generic_stereo_camera name="stereo_cam" parent="base_link" ros_topic="camera/image" cam_info_topic="camera/camera_info" update_rate="4" res_x="320" res_y="240" image_format="R8G8B8" hfov="90" baseline="0.05">
-      <origin xyz="0.05 0.0 -0.06" rpy="0 0 0"/>
+    <xacro:generic_stereo_camera name="stereo_cam" parent="base_link" ros_topic="camera/image" cam_info_topic="camera/camera_info" update_rate="20" res_x="550" res_y="500" image_format="R8G8B8" hfov="90" baseline="0.05">
+      <origin xyz="0.3 0.0 -0.06" rpy="0 0 0"/>
     </xacro:generic_stereo_camera>
 </robot>
