Commit message: Modified the launch files and added the feature of spawning the quadrotor in a different position and attitude

File: hector_quadrotor/hector_quadrotor_description/urdf/quadrotor_base.urdf.xacro (robot description, xacro)
@@ -4,13 +4,13 @@
   <xacro:property name="pi" value="3.1415926535897931" />
   <!-- Main quadrotor link -->
-  <xacro:macro name="quadrotor_base_macro">
+  <xacro:macro name="quadrotor_base_macro" params="x y z roll pitch yaw">
     <link name="base_link">
       <inertial>
         <mass value="1.477" />
-        <origin xyz="0 0 0" />
+        <origin xyz="${x} ${y} ${z}" />
         <inertia ixx="0.01152" ixy="0.0" ixz="0.0" iyy="0.01152" iyz="0.0" izz="0.0218" />
       </inertial>
       <visual>
-        <origin xyz="0 0 0" rpy="0 0 0" />
+        <origin xyz="${x} ${y} ${z}" rpy="${roll} ${pitch} ${yaw}" />
         <geometry>
           <mesh filename="package://hector_quadrotor_description/meshes/quadrotor/quadrotor_base.dae"/>
@@ -18,5 +18,5 @@
       </visual>
       <collision>
-        <origin xyz="0 0 0" rpy="0 0 0" />
+        <origin xyz="${x} ${y} ${z}" rpy="${roll} ${pitch} ${yaw}" />
         <geometry>
           <mesh filename="package://hector_quadrotor_description/meshes/quadrotor/quadrotor_base.stl"/>
@@ -24,7 +24,15 @@
       </collision>
     </link>
+    <!-- Sonar height sensor coordinates in the quadrotor frame -->
+    <xacro:property name="sonar_x_coord" value="-0.16" />
+    <xacro:property name="sonar_y_coord" value="0" />
+    <xacro:property name="sonar_z_coord" value="-0.012" />
+    <!-- Rotated sonar height sensor coordinates in the quadrotor frame -->
+    <xacro:property name="rot_sonar_x_coord" value="${(cos(yaw)*cos(pitch)*(sonar_x_coord)) + ((cos(yaw)*sin(pitch)*sin(roll)-sin(yaw)*cos(roll))*sonar_y_coord) + ((cos(yaw)*sin(pitch)*cos(roll)+sin(yaw)*sin(roll))*(sonar_z_coord))}" />
+    <xacro:property name="rot_sonar_y_coord" value="${(sin(yaw)*cos(pitch)*(sonar_x_coord)) + ((sin(yaw)*sin(pitch)*sin(roll)+cos(yaw)*cos(roll))*sonar_y_coord) + ((sin(yaw)*sin(pitch)*cos(roll)-cos(yaw)*sin(roll))*(sonar_z_coord))}" />
+    <xacro:property name="rot_sonar_z_coord" value="${(-sin(pitch)*(sonar_x_coord)) 		+  (cos(pitch)*sin(roll)*sonar_y_coord) 							 +  (cos(pitch)*cos(roll)*(sonar_z_coord))}							    " />
     <!-- Sonar height sensor -->
-    <xacro:sonar_sensor name="sonar" parent="base_link" ros_topic="sonar_height" update_rate="10" min_range="0.03" max_range="3.0" field_of_view="${40*pi/180}" ray_count="3">
-      <origin xyz="-0.16 0.0 -0.012" rpy="0 ${90*pi/180} 0"/>
+    <xacro:sonar_sensor name="sonar" parent="base_link" ros_topic="sonar_height" update_rate="10" min_range="0.03" max_range="3.0" field_of_view="${pi/4.5}" ray_count="3">
+      <origin xyz="${x+rot_sonar_x_coord} ${y+rot_sonar_y_coord} ${z+rot_sonar_z_coord}" rpy="${roll} ${(pitch)+(pi/2)} ${yaw}"/>
     </xacro:sonar_sensor>
   </xacro:macro>

File: hector_quadrotor/hector_quadrotor_description/urdf/quadrotor_with_stereo_cam_with_IMU.gazebo.xacro (robot description, xacro)
@@ -13,10 +13,10 @@
       <plugin filename="libgazebo_ros_imu_sensor.so" name="imu_plugin">
         <topicName>imu</topicName>
-        <bodyName>imu_link</bodyName>
+        <bodyName>base_link</bodyName>
         <updateRateHZ>200.0</updateRateHZ>
         <gaussianNoise>0.0</gaussianNoise>
         <xyzOffset>0 0 0</xyzOffset>
         <rpyOffset>0 0 0</rpyOffset>
-        <frameName>imu_link</frameName>
+        <frameName>base_link</frameName>
         <initialOrientationAsReference>false</initialOrientationAsReference>
       </plugin>

File: hector_quadrotor/hector_quadrotor_description/urdf/quadrotor_with_stereo_cam_with_IMU.urdf.xacro (robot description, xacro)
@@ -2,12 +2,27 @@
 <robot name="quadrotor" xmlns:xacro="http://www.ros.org/wiki/xacro">
     <xacro:property name="M_PI" value="3.1415926535897931" />
+    <!-- Desired quadrotor position and attitude -->
+    <xacro:property name="X" value="0" />
+    <xacro:property name="Y" value="0" />
+    <xacro:property name="Z" value="0" />
+    <xacro:property name="ROLL" value="${0 * pi/180}" />
+    <xacro:property name="PITCH" value="${0 * pi/180}" />
+    <xacro:property name="YAW" value="${0 * pi/180}" />
+    <!-- Camera coordinates in the quadrotor frame -->
+    <xacro:property name="camera_x_coord" value="0.3" />
+    <xacro:property name="camera_y_coord" value="0" />
+    <xacro:property name="camera_z_coord" value="-0.06" />
+    <!-- Rotated camera coordinates in the quadrotor frame -->
+    <xacro:property name="rot_camera_x_coord" value="${(cos(YAW)*cos(PITCH)*(camera_x_coord)) + ((cos(YAW)*sin(PITCH)*sin(ROLL)-sin(YAW)*cos(ROLL))*camera_y_coord) + ((cos(YAW)*sin(PITCH)*cos(ROLL)+sin(YAW)*sin(ROLL))*(camera_z_coord))}" />
+    <xacro:property name="rot_camera_y_coord" value="${(sin(YAW)*cos(PITCH)*(camera_x_coord)) + ((sin(YAW)*sin(PITCH)*sin(ROLL)+cos(YAW)*cos(ROLL))*camera_y_coord) + ((sin(YAW)*sin(PITCH)*cos(ROLL)-cos(YAW)*sin(ROLL))*(camera_z_coord))}" />
+    <xacro:property name="rot_camera_z_coord" value="${(-sin(PITCH)*(camera_x_coord)) 		  +  (cos(PITCH)*sin(ROLL)*camera_y_coord) 								+  (cos(PITCH)*cos(ROLL)*(camera_z_coord))}							    " />
     <!-- Included URDF Files -->
     <xacro:include filename="$(find hector_quadrotor_description)/urdf/quadrotor_base.urdf.xacro" />
-    <!-- Instantiate quadrotor_base_macro once (has no parameters atm) -->
-    <xacro:quadrotor_base_macro />
+    <!-- Instantiate quadrotor_base_macro once -->
+    <xacro:quadrotor_base_macro x="${X}" y="${Y}" z="${Z}" roll="${ROLL}" pitch="${PITCH}" yaw="${YAW}"/>
     <!-- Stereo camera -->
     <xacro:include filename="$(find hector_sensors_description)/urdf/generic_stereo_camera.urdf.xacro" />
     <xacro:generic_stereo_camera name="stereo_cam" parent="base_link" ros_topic="camera/image" cam_info_topic="camera/camera_info" update_rate="20" res_x="550" res_y="500" image_format="R8G8B8" hfov="90" baseline="0.05">
-      <origin xyz="0.3 0.0 -0.06" rpy="0 0 0"/>
+      <origin xyz="${X+rot_camera_x_coord} ${Y+rot_camera_y_coord} ${Z+rot_camera_z_coord}" rpy="${ROLL} ${PITCH} ${YAW}"/>
     </xacro:generic_stereo_camera>
 </robot>

Commit message: Fixed the problems with spawning the quadrotor anywhere, updated launch files, added missing ones and fixed a bug in the outdoor world

File: hector_quadrotor/hector_quadrotor_description/urdf/quadrotor_base.urdf.xacro (robot description, xacro)
@@ -4,13 +4,13 @@
   <xacro:property name="pi" value="3.1415926535897931" />
   <!-- Main quadrotor link -->
-  <xacro:macro name="quadrotor_base_macro" params="x y z roll pitch yaw">
+  <xacro:macro name="quadrotor_base_macro">
     <link name="base_link">
       <inertial>
         <mass value="1.477" />
-        <origin xyz="${x} ${y} ${z}" />
+        <origin xyz="0 0 0" />
         <inertia ixx="0.01152" ixy="0.0" ixz="0.0" iyy="0.01152" iyz="0.0" izz="0.0218" />
       </inertial>
       <visual>
-        <origin xyz="${x} ${y} ${z}" rpy="${roll} ${pitch} ${yaw}" />
+        <origin xyz="0 0 0" rpy="0 0 0" />
         <geometry>
           <mesh filename="package://hector_quadrotor_description/meshes/quadrotor/quadrotor_base.dae"/>
@@ -18,5 +18,5 @@
       </visual>
       <collision>
-        <origin xyz="${x} ${y} ${z}" rpy="${roll} ${pitch} ${yaw}" />
+        <origin xyz="0 0 0" rpy="0 0 0" />
         <geometry>
           <mesh filename="package://hector_quadrotor_description/meshes/quadrotor/quadrotor_base.stl"/>
@@ -29,10 +29,10 @@
     <xacro:property name="sonar_z_coord" value="-0.012" />
     <!-- Rotated sonar height sensor coordinates in the quadrotor frame -->
-    <xacro:property name="rot_sonar_x_coord" value="${(cos(yaw)*cos(pitch)*(sonar_x_coord)) + ((cos(yaw)*sin(pitch)*sin(roll)-sin(yaw)*cos(roll))*sonar_y_coord) + ((cos(yaw)*sin(pitch)*cos(roll)+sin(yaw)*sin(roll))*(sonar_z_coord))}" />
+    <!--<xacro:property name="rot_sonar_x_coord" value="${(cos(yaw)*cos(pitch)*(sonar_x_coord)) + ((cos(yaw)*sin(pitch)*sin(roll)-sin(yaw)*cos(roll))*sonar_y_coord) + ((cos(yaw)*sin(pitch)*cos(roll)+sin(yaw)*sin(roll))*(sonar_z_coord))}" />
     <xacro:property name="rot_sonar_y_coord" value="${(sin(yaw)*cos(pitch)*(sonar_x_coord)) + ((sin(yaw)*sin(pitch)*sin(roll)+cos(yaw)*cos(roll))*sonar_y_coord) + ((sin(yaw)*sin(pitch)*cos(roll)-cos(yaw)*sin(roll))*(sonar_z_coord))}" />
-    <xacro:property name="rot_sonar_z_coord" value="${(-sin(pitch)*(sonar_x_coord)) 		+  (cos(pitch)*sin(roll)*sonar_y_coord) 							 +  (cos(pitch)*cos(roll)*(sonar_z_coord))}							    " />
+    <xacro:property name="rot_sonar_z_coord" value="${(-sin(pitch)*(sonar_x_coord)) 		+  (cos(pitch)*sin(roll)*sonar_y_coord) 							 +  (cos(pitch)*cos(roll)*(sonar_z_coord))}							    " />-->
     <!-- Sonar height sensor -->
     <xacro:sonar_sensor name="sonar" parent="base_link" ros_topic="sonar_height" update_rate="10" min_range="0.03" max_range="3.0" field_of_view="${pi/4.5}" ray_count="3">
-      <origin xyz="${x+rot_sonar_x_coord} ${y+rot_sonar_y_coord} ${z+rot_sonar_z_coord}" rpy="${roll} ${(pitch)+(pi/2)} ${yaw}"/>
+      <origin xyz="${sonar_x_coord} ${sonar_y_coord} ${sonar_z_coord}" rpy="0 ${pi/2} 0"/>
     </xacro:sonar_sensor>
   </xacro:macro>

File: hector_quadrotor/hector_quadrotor_description/urdf/quadrotor_with_stereo_cam_with_IMU.urdf.xacro (robot description, xacro)
@@ -2,11 +2,11 @@
 <robot name="quadrotor" xmlns:xacro="http://www.ros.org/wiki/xacro">
     <xacro:property name="M_PI" value="3.1415926535897931" />
-    <!-- Desired quadrotor position and attitude -->
-    <xacro:property name="X" value="0" />
+    <!-- The quadrotor position and attitude, equal to the one in the launch file -->
+    <!--<xacro:property name="X" value="0" />
     <xacro:property name="Y" value="0" />
     <xacro:property name="Z" value="0" />
     <xacro:property name="ROLL" value="${0 * pi/180}" />
     <xacro:property name="PITCH" value="${0 * pi/180}" />
-    <xacro:property name="YAW" value="${0 * pi/180}" />
+    <xacro:property name="YAW" value="${0 * pi/180}" />-->
     <!-- Camera coordinates in the quadrotor frame -->
     <xacro:property name="camera_x_coord" value="0.3" />
@@ -14,15 +14,15 @@
     <xacro:property name="camera_z_coord" value="-0.06" />
     <!-- Rotated camera coordinates in the quadrotor frame -->
-    <xacro:property name="rot_camera_x_coord" value="${(cos(YAW)*cos(PITCH)*(camera_x_coord)) + ((cos(YAW)*sin(PITCH)*sin(ROLL)-sin(YAW)*cos(ROLL))*camera_y_coord) + ((cos(YAW)*sin(PITCH)*cos(ROLL)+sin(YAW)*sin(ROLL))*(camera_z_coord))}" />
+    <!--<xacro:property name="rot_camera_x_coord" value="${(cos(YAW)*cos(PITCH)*(camera_x_coord)) + ((cos(YAW)*sin(PITCH)*sin(ROLL)-sin(YAW)*cos(ROLL))*camera_y_coord) + ((cos(YAW)*sin(PITCH)*cos(ROLL)+sin(YAW)*sin(ROLL))*(camera_z_coord))}" />
     <xacro:property name="rot_camera_y_coord" value="${(sin(YAW)*cos(PITCH)*(camera_x_coord)) + ((sin(YAW)*sin(PITCH)*sin(ROLL)+cos(YAW)*cos(ROLL))*camera_y_coord) + ((sin(YAW)*sin(PITCH)*cos(ROLL)-cos(YAW)*sin(ROLL))*(camera_z_coord))}" />
-    <xacro:property name="rot_camera_z_coord" value="${(-sin(PITCH)*(camera_x_coord)) 		  +  (cos(PITCH)*sin(ROLL)*camera_y_coord) 								+  (cos(PITCH)*cos(ROLL)*(camera_z_coord))}							    " />
+    <xacro:property name="rot_camera_z_coord" value="${(-sin(PITCH)*(camera_x_coord)) 		  +  (cos(PITCH)*sin(ROLL)*camera_y_coord) 								+  (cos(PITCH)*cos(ROLL)*(camera_z_coord))}							    " />-->
     <!-- Included URDF Files -->
     <xacro:include filename="$(find hector_quadrotor_description)/urdf/quadrotor_base.urdf.xacro" />
     <!-- Instantiate quadrotor_base_macro once -->
-    <xacro:quadrotor_base_macro x="${X}" y="${Y}" z="${Z}" roll="${ROLL}" pitch="${PITCH}" yaw="${YAW}"/>
+    <xacro:quadrotor_base_macro/>
     <!-- Stereo camera -->
     <xacro:include filename="$(find hector_sensors_description)/urdf/generic_stereo_camera.urdf.xacro" />
     <xacro:generic_stereo_camera name="stereo_cam" parent="base_link" ros_topic="camera/image" cam_info_topic="camera/camera_info" update_rate="20" res_x="550" res_y="500" image_format="R8G8B8" hfov="90" baseline="0.05">
-      <origin xyz="${X+rot_camera_x_coord} ${Y+rot_camera_y_coord} ${Z+rot_camera_z_coord}" rpy="${ROLL} ${PITCH} ${YAW}"/>
+      <origin xyz="${camera_x_coord} ${camera_y_coord} ${camera_z_coord}" rpy="0 0 0"/>
     </xacro:generic_stereo_camera>
 </robot>

Commit message: Modified some launch files and added an hokuyo laser to the drone

File: hector_quadrotor/hector_quadrotor_description/urdf/quadrotor_base.urdf.xacro (robot description, xacro)
@@ -28,8 +28,4 @@
     <xacro:property name="sonar_y_coord" value="0" />
     <xacro:property name="sonar_z_coord" value="-0.012" />
-    <!-- Rotated sonar height sensor coordinates in the quadrotor frame -->
-    <!--<xacro:property name="rot_sonar_x_coord" value="${(cos(yaw)*cos(pitch)*(sonar_x_coord)) + ((cos(yaw)*sin(pitch)*sin(roll)-sin(yaw)*cos(roll))*sonar_y_coord) + ((cos(yaw)*sin(pitch)*cos(roll)+sin(yaw)*sin(roll))*(sonar_z_coord))}" />
-    <xacro:property name="rot_sonar_y_coord" value="${(sin(yaw)*cos(pitch)*(sonar_x_coord)) + ((sin(yaw)*sin(pitch)*sin(roll)+cos(yaw)*cos(roll))*sonar_y_coord) + ((sin(yaw)*sin(pitch)*cos(roll)-cos(yaw)*sin(roll))*(sonar_z_coord))}" />
-    <xacro:property name="rot_sonar_z_coord" value="${(-sin(pitch)*(sonar_x_coord)) 		+  (cos(pitch)*sin(roll)*sonar_y_coord) 							 +  (cos(pitch)*cos(roll)*(sonar_z_coord))}							    " />-->
     <!-- Sonar height sensor -->
     <xacro:sonar_sensor name="sonar" parent="base_link" ros_topic="sonar_height" update_rate="10" min_range="0.03" max_range="3.0" field_of_view="${pi/4.5}" ray_count="3">

File: hector_quadrotor/hector_quadrotor_description/urdf/quadrotor_with_stereo_cam_with_hokuyo.gazebo.xacro (robot description, xacro)
@@ -1,5 +1,5 @@
 <?xml version="1.0"?>
 <robot name="quadrotor" xmlns:xacro="http://www.ros.org/wiki/xacro">
-    <xacro:include filename="$(find hector_quadrotor_description)/urdf/quadrotor_with_stereo_cam_with_IMU.urdf.xacro" />
+    <xacro:include filename="$(find hector_quadrotor_description)/urdf/quadrotor_with_stereo_cam_with_hokuyo.urdf.xacro" />
     <xacro:include filename="$(find hector_quadrotor_gazebo)/urdf/quadrotor_plugins.gazebo.xacro" />
     <!-- Add the IMU to the base link -->
